File: BD35F-FridgeController/BD35F-FridgeController.kicad_pcb (KiCad board)
At the start: 2 copper layers, 44.8 x 64.8 mm, 9 parts, among them J1 12 Volt, J2 DS18B20, J3 BD35F, Q1 BC337, U1 WeMos_D1_mini, U2 R-78E50-10_TO220

Commit message: Add files via upload
Parts:
- added C1: 10 µF, Capacitor_THT:CP_Radial_D5.0mm_P2.50mm, F.Cu at (85.9, 84.8)
- moved Q1 2.77 mm to (94.6, 84.9)
Routing:
- net Net-(D1-K): track 35.0 -> 41.8 mm
- net Net-(Q1-B): track 16.8 -> 10.6 mm
- net GND: track 130.8 -> 136.7 mm
- net Net-(J3-Pin_1): track 12.2 -> 9.52 mm
- net Net-(U1-MISO/D6): track 20.6 -> 22.8 mm
Other:
- board text added: "BD35F Fridge Control Version 1.1"
- board text removed: "BD35F Fridge Control Version 1.0"
