File: BD35F-FridgeController/BD35F-FridgeController.kicad_sch (KiCad schematic)
At the start: 9 parts, among them J1 12 Volt, J2 DS18B20, J3 BD35F, Q1 BC337, U1 WeMos_D1_mini, U2 R-78E50-10_TO220

Commit message: Add files via upload
Parts:
- added C1: 10 µF, Capacitor_THT:CP_Radial_D5.0mm_P2.50mm, symbol Device:C_Polarized
Connections:
- net GND: now also C1.2
- net at D1.1 (K), U2.1 (VI): now also C1.1
Changed lines of the file:
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@@
 	(paper "A4")
+	(junction
+		(at 59.69 63.5)
+		(diameter 0)
+		(color 0 0 0 0)
+	)
 	(junction
 		(at 71.12 71.12)
@@
 	)
 	(junction
+		(at 59.69 71.12)
+		(diameter 0)
+		(color 0 0 0 0)
+	)
+	(junction
 		(at 87.63 130.81)
 		(diameter 0)
@@
 	(wire
 		(pts
+			(xy 59.69 63.5) (xy 63.5 63.5)
+		)
+		(stroke
+			(width 0)
+			(type default)
+		)
+	)
+	(wire
+		(pts
 			(xy 82.55 76.2) (xy 125.73 76.2)
 		)
@@
 	(wire
 		(pts
+			(xy 59.69 71.12) (xy 71.12 71.12)
+		)
+		(stroke
+			(width 0)
+			(type default)
+		)
+	)
+	(wire
+		(pts
 			(xy 46.99 83.82) (xy 46.99 76.2)
 		)
@@
 	(wire
 		(pts
-			(xy 58.42 63.5) (xy 63.5 63.5)
+			(xy 58.42 63.5) (xy 59.69 63.5)
 		)
 		(stroke
@@
 	(wire
 		(pts
-			(xy 46.99 71.12) (xy 71.12 71.12)
+			(xy 46.99 71.12) (xy 59.69 71.12)
 		)
 		(stroke
@@
 					(unit 1)
 				)
+			)
+		)
+	)
+	(symbol
+		(lib_id "Device:C_Polarized")
+		(at 59.69 67.31 0)
+		(unit 1)
+		(exclude_from_sim no)
+		(in_bom yes)
+		(on_board yes)
+		(dnp no)
+		(property "Reference" "C1"
+			(at 53.34 67.564 0)
+			(effects
+				(font
+					(size 1.27 1.27)
+				)
+				(justify left)
+			)
+		)
+		(property "Value" "10 µF"
+			(at 51.816 69.85 0)
+			(effects
+				(font
+					(size 1.27 1.27)
+				)
+				(justify left)
+			)
+		)
+		(property "Footprint" "Capacitor_THT:CP_Radial_D5.0mm_P2.50mm"
+			(at 60.6552 71.12 0)
+			(effects
+				(font
+					(size 1.27 1.27)
+				)
+				(hide yes)
+			)
+		)
+		(property "Datasheet" "~"
+			(at 59.69 67.31 0)
+			(effects
+				(font
+					(size 1.27 1.27)
+				)
+				(hide yes)
+			)
+		)
+		(property "Description" "Polarized capacitor"
+			(at 59.69 67.31 0)
+			(effects
+				(font
+					(size 1.27 1.27)
+				)
+				(hide yes)
+			)
+		)
+		(pin "1"
+		)
+		(pin "2"
+		)
+		(instances
+			(project "BD35F-FridgeController"
+				(path "/949c3da7-86cf-42b3-9a90-86860601a60c"
+					(reference "C1")
+					(unit 1)
+				)
